File: lna_fm_98mhz.kicad_pcb (KiCad board)
At the start: 2 copper layers, 46 x 30 mm, 30 parts, among them J1 SMA_50R_IN, J2 SMA_50R_OUT, J3 BAT_PADS, Q1 MMBT5179

Commit message: Implement input bandpass pre-filter merged with input matching network
- Merged parallel LC tank (L1=18nH || C2=47pF) at 50-ohm RF input with series C1=100pF DC block to emitter.
- Suppresses out-of-band signals (<88 MHz shunted by L1, >108 MHz shunted by C2) while providing exact step-down transformation to low-impedance common-base emitter.
- Preserves 98 MHz center performance: S21 = +19.88 dB, S11 = -22.27 dB (VSWR 1.17:1), Zin = 43.1 - j1.9 Ohm.
- Updated Qucs simulation netlists, Touchstone s2p, and schematic generator scripts.
- Updated KiCad schematic, zero ERC violations.
- Synthesized PCB layout with C2 placed and routed, zero DRC errors.
- Regenerated production Gerbers, Excellon drill files, 3D STEP model, and 2D/3D visual renders.
- Updated README.md and AGENT.md documentation and BOM.
Parts:
- added C2: 47pF, C_0603_1608Metric, F.Cu at (6.50, 17.5)
- L1: value 27nH -> 18nH
Routing:
- net GND: track 23.3 -> 25.0 mm
- net /RF_IN_50R: track 10.6 -> 12.3 mm

Commit message: Optimize input matching network for -31.87 dB return loss at 98 MHz
- Parameter optimization: L1=22nH (0603 E12), C2=27pF (0603 E12), C1=91pF (0805 E24).
- Restores real input resistance to 52.5 Ohm (from 43.1 Ohm) by tuning C1 transformation Q.
- Improves S11 return loss from -22.27 dB to -31.87 dB (VSWR 1.05:1).
- Preserves high gain (S21 = +19.91 dB) and out-of-band rejection (-19.9 dB at 50 MHz, +2.1 dB at 200 MHz).
- Updated Qucs netlists, Touchstone s2p, and schematic generators.
- Regenerated KiCad schematic and PCB layout with 0 ERC / 0 DRC violations.
- Regenerated production Gerbers, Excellon drills, 3D STEP model, and 2D/3D renders.
- Updated README.md, AGENT.md, and PRE_FILTER_COMPARISON.md.
Parts:
- C1: value 100pF -> 91pF
- C2: value 47pF -> 27pF
- L1: value 18nH -> 22nH
